File: hardware/interstate/_autosave-interstate.kicad_pcb (KiCad board)
At the start: 4 copper layers, 125 x 125 mm, 153 parts, among them J1 Lamp 1 Out, J10 CAN, J11 ESC1_PWR, J12 ESC1_CTRL, J13 ESC1_SW, J14 ESC2_PWR, J15 ESC2_CTRL, J16 ESC2_SW, J17 ESC3_PWR, J18 ESC3_CTRL, J19 ESC3_SW, J2 ESTOP1, J20 SWD, J3 ESTOP2, J4 Lamp 3 Out, J5 Lamp 2 Out, J6 Lamp 4 Out, J7 Conn_01x02, J8 RJ45, J9 RJ45, Q1 2N7002, Q2 2N7002, Q3 2N7002, Q4 2N7002, Q5 Q_NMOS_GDS, Q6 2N7002, Q7 2N7002, Q8 2N7002, SW1 RST, U1 LM339, U2 VCB4824SBO, U3 MCP1792T, U4 MCP1804x-3302xMT, U5 SHHD001A3B41Z, U6 LT1641-1, U7 SN65HVD232, U9 STM32F334R8Tx

Commit message: routing first try
Routing:
- net +3V3: track 131.9 -> 133.6 mm, vias 12 -> 13
Changed lines of the file:
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@@
   (segment (start 145.542 92.202) (end 145.542 101.727) (width 1) (layer "F.Cu") (net 44))
   (segment (start 120.625 134.391) (end 120.904 134.112) (width 0.254) (layer "F.Cu") (net 44))
+  (segment (start 126.875 147.675) (end 126.875 149.227) (width 0.254) (layer "F.Cu") (net 44))
   (segment (start 125.875 135.25) (end 123.625 133) (width 0.254) (layer "F.Cu") (net 44))
   (segment (start 146.46 149) (end 146.812 149.352) (width 0.254) (layer "F.Cu") (net 44))
@@
   (segment (start 154.882 102.05) (end 154.813 101.981) (width 0.254) (layer "F.Cu") (net 44))
   (segment (start 158.525 102.135) (end 156.085 102.135) (width 0.254) (layer "F.Cu") (net 44))
+  (segment (start 126.875 149.227) (end 127 149.352) (width 0.254) (layer "F.Cu") (net 44))
   (segment (start 149 88.744) (end 145.542 92.202) (width 1) (layer "F.Cu") (net 44))
   (segment (start 133.375 147.675) (end 134.675 147.675) (width 0.254) (layer "F.Cu") (net 44))
@@
   (segment (start 61.175 90) (end 60 90) (width 0.508) (layer "F.Cu") (net 44))
   (via (at 122.428 133.604) (size 0.8) (drill 0.4) (layers "F.Cu" "B.Cu") (net 44))
+  (via (at 127 149.352) (size 0.8) (drill 0.4) (layers "F.Cu" "B.Cu") (net 44))
   (via (at 121 147) (size 0.8) (drill 0.4) (layers "F.Cu" "B.Cu") (free) (net 44))
   (via (at 146.812 149.352) (size 0.8) (drill 0.4) (layers "F.Cu" "B.Cu") (net 44))
