File: hardware/interstate/interstate.kicad_pcb (KiCad board)
At the start: 4 copper layers, 125 x 125 mm, 153 parts, among them J1 Lamp 1 Out, J10 CAN, J11 ESC1_PWR, J12 ESC1_CTRL, J13 ESC1_SW, J14 ESC2_PWR, J15 ESC2_CTRL, J16 ESC2_SW, J17 ESC3_PWR, J18 ESC3_CTRL, J19 ESC3_SW, J2 ESTOP1, J20 SWD, J3 ESTOP2, J4 Lamp 3 Out, J5 Lamp 2 Out, J6 Lamp 4 Out, J7 Conn_01x02, J8 RJ45, J9 RJ45, Q1 2N7002, Q2 2N7002, Q3 2N7002, Q4 2N7002, Q5 Q_NMOS_GDS, Q6 2N7002, Q7 2N7002, Q8 2N7002, SW1 RST, U1 LM339, U2 VCB4824SBO, U3 MCP1792T, U4 MCP1804x-3302xMT, U5 SHHD001A3B41Z, U6 LT1641-1, U7 SN65HVD232, U9 STM32F334R8Tx

Commit message: More routing work - changed some MCU pinout
Parts:
- moved R16 53.8 mm to (156.0, 138.2), turned to -90 degrees
- moved R15 51.0 mm to (154.6, 138.2), turned to -90 degrees
- moved C5 49.3 mm to (154.1, 141.2), turned to 0 degrees
- moved U3 45.9 mm to (152.1, 147.2), turned to -90 degrees
- moved C18 42.4 mm to (103.5, 137.6)
- moved R50 42.4 mm to (103.5, 139.2)
- moved SW1 42.4 mm to (106.8, 133.2)
- moved C7 42.2 mm to (150.6, 141.2), turned to 180 degrees
- moved R11 10.9 mm to (157.0, 72.8)
- moved R12 10.9 mm to (157.0, 75.8)
- moved R8 10.9 mm to (157.0, 74.2)
- moved C1 9.62 mm to (168.8, 83.8), turned to 0 degrees
- moved R42 8.40 mm to (161.8, 75.8)
- moved R43 8.40 mm to (161.8, 74.2)
- moved R45 7.40 mm to (161.8, 83.0)
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Connections:
- U1 pad 1: Net-(R45-Pad1) -> GND
- U1 pad 10: GND -> Net-(R41-Pad2)
- U1 pad 11: GND -> Net-(R40-Pad2)
- U1 pad 13: GND -> Net-(R44-Pad1)
- U1 pad 14: GND -> Net-(R45-Pad1)
- U1 pad 2: Net-(R44-Pad1) -> GND
- U1 pad 4: Net-(R41-Pad2) -> GND
- U1 pad 5: Net-(R40-Pad2) -> GND
- U1 pad 6: Net-(R43-Pad2) -> GND
- U1 pad 7: Net-(R42-Pad2) -> GND
- U1 pad 8: GND -> Net-(R43-Pad2)
- U1 pad 9: GND -> Net-(R42-Pad2)
- U9 pad 14: unconnected-(U9-Pad14) -> /ESC1_ON
- U9 pad 15: /ESC2_ADC1_UNFILT -> /ESC1_ADC2_UNFILT
- U9 pad 16: /ESC2_P -> /ESC1_P
- U9 pad 17: /ESC2_N -> /ESC1_N
- U9 pad 20: /ESC2_ADC2_UNFILT -> /ESC1_ADC1_UNFILT
- U9 pad 21: /ESC2_ON -> /ESC3_ON
- U9 pad 22: unconnected-(U9-Pad22) -> /ESC3_ADC2_UNFILT
- U9 pad 23: /ESC1_ADC1_UNFILT -> unconnected-(U9-Pad23)
- U9 pad 24: /ESC1_P -> /ESC3_P
- U9 pad 25: /ESC1_N -> /ESC3_N
- U9 pad 26: /ESC1_ADC2_UNFILT -> /ESC3_ADC1_UNFILT
- U9 pad 27: /ESC1_ON -> /ESC2_ADC2_UNFILT
- U9 pad 29: /ESC3_P -> /ESC2_P
- U9 pad 30: /ESC3_N -> /ESC2_N
- U9 pad 34: /ESC3_ON -> unconnected-(U9-Pad34)
- U9 pad 35: /ESC3_ADC1_UNFILT -> /ESC2_ADC1_UNFILT
- U9 pad 36: /ESC3_ADC2_UNFILT -> /ESC2_ON
Routing:
- net +12V: track 109.3 -> 9.96 mm, vias 3 -> 2
- net +3V3: track 131.9 -> 43.6 mm, vias 12 -> 9
- net +24V: track 61.2 -> 4.71 mm
- net /ESC2_ON: track 2.08 -> 48.5 mm
- net /nESTOP1: track 2.60 -> 38.9 mm
- net /ESC1_ADC1_UNFILT: track 33.3 -> 68.9 mm
- net /ESC2_ADC2_UNFILT: track 8.85 -> 41.7 mm
- net /nESTOP2: track 0.00 -> 32.4 mm
- net /ESC2_P: track 11.7 -> 43.1 mm, vias 0 -> 2
- net /ESC1_N: track 41.7 -> 72.9 mm, vias 0 -> 2
- net /ESC2_N: track 11.7 -> 42.8 mm
- net /ESC2_ADC1_UNFILT: track 4.32 -> 34.8 mm
- net /ESC1_P: track 41.7 -> 72.1 mm
- net /ESC1_ON: track 50.0 -> 79.5 mm
- net /ESC1_ADC2_UNFILT: track 36.0 -> 64.6 mm
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- added copper zone on F.Cu, net GND
- removed copper zone on F.Cu, net +3V3
Other:
- board text added: "ESC1"
- board text added: "ESC2"
- board text added: "ESC3"

Commit message: finished routing v1?
Parts:
- removed U2: VCB4824SBO, interstate_footprints:VCB4824SB0-30WR3
- added 12V: TestPoint_Pad_D1.0mm, TestPoint:TestPoint_Pad_D1.0mm, F.Cu at (141.1, 93.5)
- added 24V: TestPoint_Pad_D1.0mm, TestPoint:TestPoint_Pad_D1.0mm, F.Cu at (141.1, 103.7)
- added 24V CONVERTER: VCB4824SBO, interstate_footprints:VCB4824SB0-30WR3, F.Cu at (120.0, 113.1)
- added FB: TestPoint_Pad_D1.0mm, TestPoint:TestPoint_Pad_D1.0mm, F.Cu at (61.6, 92.5)
- added G***: LOGO, interstate_footprints:paradigm_ss, F.Cu at (93.9, 126.3)
- added REF**: TestPoint_Pad_D1.0mm, TestPoint:TestPoint_Pad_D1.0mm, F.Cu at (144.1, 64.3)
- added SYS_ON: TestPoint_Pad_D1.0mm, TestPoint:TestPoint_Pad_D1.0mm, F.Cu at (60.6, 83.6)
- added nESTOP2: TestPoint_Pad_D1.0mm, TestPoint:TestPoint_Pad_D1.0mm, F.Cu at (153.5, 59.2)
- 12V CONVERTER: renamed from U5
- moved R30 88.6 mm to (140.0, 132.2), turned to 90 degrees
- moved D2 85.2 mm to (102.6, 136.9), turned to 0 degrees
- moved D3 82.0 mm to (102.6, 133.9), turned to 0 degrees
- moved R46 79.2 mm to (106.3, 136.9), turned to 180 degrees
- moved R47 75.8 mm to (106.3, 133.9), turned to 180 degrees
- moved R28 18.7 mm to (76.2, 102.6), turned to 90 degrees
- moved C18 12.1 mm to (107.3, 149.1), turned to 180 degrees
- moved R50 12.0 mm to (107.3, 150.6), turned to 0 degrees
- moved RESET 11.6 mm to (104.3, 144.6)
- moved R4 8.49 mm to (159.5, 57.8)
- moved R5 8.49 mm to (157.5, 57.8)
- moved C4 2.37 mm to (163.9, 67.1), turned to 0 degrees
- moved R23 2.30 mm to (138.0, 114.7)
- moved R14 2.17 mm to (159.5, 66.3)
- moved R16 1.68 mm to (154.3, 138.2)
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- renumbered J10 to CAN, J11 to ESC1-POWER, J13 to ESC1-SW, J12 to ESC1_SIGNAL, J17 to ESC2-POWER, J15 to ESC2-SIGNAL, J16 to ESC2-SW, J14 to ESC3-POWER, J19 to ESC3-SW, J18 to ESC3_SIGNAL, J2 to ESTOP1, J3 to ESTOP2, J1 to LAMP1, J5 to LAMP2, J4 to LAMP3, J6 to LAMP4, J8 to PASSIVE-ETH, J7 to POWER-IN, J9 to POWERED-ETH, SW1 to RESET, J20 to SWD
Connections:
- ESTOP2 pad 1: Net-(J3-Pad1) -> GND
- ESTOP2 pad 2: /ESTOP2 -> /nESTOP2
- ESTOP2 pad 3: /nESTOP2 -> /ESTOP2
- ESTOP2 pad 4: GND -> Net-(R4-Pad2)
- R4 pad 2: Net-(J3-Pad1) -> Net-(R4-Pad2)
- R5 pad 2: Net-(J3-Pad1) -> Net-(R4-Pad2)
- R54 pad 1: /ESC1_GND -> GND
- R61 pad 1: /ESC2_GND -> GND
- R68 pad 1: /ESC3_GND -> GND
- U9 pad 2: unconnected-(U9-Pad2) -> /LAMP3_ON
- U9 pad 3: unconnected-(U9-Pad3) -> /LAMP2_ON
- U9 pad 4: unconnected-(U9-Pad4) -> /LAMP1_ON
- U9 pad 43: unconnected-(U9-Pad43) -> /BATT_GOOD
- U9 pad 5: unconnected-(U9-Pad5) -> /LED1
- U9 pad 6: unconnected-(U9-Pad6) -> /LED2
- U9 pad 62: unconnected-(U9-Pad62) -> /LAMP4_ON
Routing:
- net /BATT_GOOD: track 2.76 -> 139.1 mm, vias 0 -> 4
- net +12V: track 9.96 -> 134.8 mm, vias 2 -> 7
- net /LAMP1_ON: track 2.18 -> 114.0 mm, vias 0 -> 2
- net /SYS_ON: track 6.80 -> 118.1 mm, vias 0 -> 4
- net /LAMP2_ON: track 2.08 -> 102.8 mm, vias 0 -> 2
- net +3V3: track 43.6 -> 142.2 mm, vias 9 -> 19
- net /LAMP4_ON: track 2.11 -> 90.0 mm, vias 0 -> 2
- net /LAMP3_ON: track 2.08 -> 89.9 mm, vias 0 -> 2
- net /nRESET: track 10.2 -> 84.9 mm
- net +24V: track 4.71 -> 73.7 mm, vias 2 -> 4
- net GND: track 78.4 -> 109.7 mm, vias 43 -> 103
- net Net-(C30-Pad1): track 6.26 -> 30.5 mm, vias 1 -> 0
- net /LED1: track 0.00 -> 21.0 mm
- net +5V: track 2.55 -> 21.8 mm
- net /LED2: track 0.00 -> 18.4 mm
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- added copper zone on F.Cu, net +3V3
- added copper zone on F.Cu, net +5V
- added copper zone on B.Cu, net /BATT_PROT
- added copper zone on B.Cu, net GND
- added copper zone on In2.Cu, net GND
- added copper zone on F.Cu, net Net-(C4-Pad1)
Other:
- board text added: "Francis Walsh 2022"
- board text removed: "ESC1"
- board text removed: "ESC2"
- board text removed: "ESC3"
