File: hardware/interstate/interstate.kicad_sch (KiCad schematic)
At the start: 154 parts, among them J1 Lamp 1 Out, J10 CAN, J11 ESC1_PWR, J12 ESC1_CTRL, J13 ESC1_SW, J14 ESC2_PWR, J15 ESC2_CTRL, J16 ESC2_SW, J17 ESC3_PWR, J18 ESC3_CTRL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

Commit message: routing first try
Parts:
- added C28, C29, C30: 10nF, Capacitor_SMD:C_0603_1608Metric, symbol Device:C_Small
- gave numbers to parts that had none: 1
Connections:
- net CAN_TX is gone; now on net CAN_P: R75.1, U9.45 (PA12)
- net BATT_PROT: now also C2.1, C3.1, U2.1 (VIN), U5.1 (VIN+)
- net BATT_RAW: now also C29.1; no longer C2.1, C3.1, U2.1 (VIN), U5.1 (VIN+)
- net CAN_P: no longer J10.2 (Pin_2), R48.1, U7.7 (CANH)
- net GND: now also C28.2, C29.2, C30.2
- net SYS_ON: now also C28.1
- net at R28.2, R29.1, U6.2 (FB): now also C30.1
- net CAN_L renamed CAN-
- net CAN_RX renamed CAN_N
- net ESC1_RX renamed ESC1_N
- net ESC1_TX renamed ESC1_P
- net ESC2_RX renamed ESC2_N
- net ESC2_TX renamed ESC2_P
- net ESC3_RX renamed ESC3_N
- net ESC3_TX renamed ESC3_P
- new net CAN+: J10.2 (Pin_2), R48.1, U7.7 (CANH)
- no-connect marks 26 -> 27
Other:
- note added: "CAN_P = CAN_TX CAN_N = CAN_RX"
- note added: "ESC_P = ESC_TX ESC_N = ESC_RX"
- moved on the sheet: R30

Commit message: More routing work - changed some MCU pinout
Parts:
- C19: value (none) -> 0.1uF; footprint (none) -> Capacitor_SMD:C_0805_2012Metric
- C2: value (none) -> 33uF; footprint (none) -> Capacitor_THT:CP_Radial_D8.0mm_P3.50mm
- C25: value (none) -> 4.7uF
- C3: value (none) -> 100uF; footprint (none) -> Capacitor_THT:CP_Radial_D10.0mm_P5.00mm
- C5, C7: value (none) -> 2.2uF; footprint (none) -> Capacitor_SMD:C_0805_2012Metric
- C9: value (none) -> 4.7uF; footprint (none) -> Capacitor_SMD:C_0805_2012Metric
- H1, H2, H3, H4: value (none) -> M3; footprint (none) -> MountingHole:MountingHole_3.2mm_M3_Pad_Via
- J20: value (none) -> SWD; footprint (none) -> Connector_PinSocket_1.27mm:PinSocket_2x03_P1.27mm_Vertical
- J9: value (none) -> RJ45; footprint (none) -> Connector_RJ:RJ45_Amphenol_54602-x08_Horizontal
- Q5: value (none) -> Q_NMOS_GDS; footprint (none) -> Package_TO_SOT_SMD:TO-263-2
- R21: value (none) -> 1; footprint (none) -> Resistor_SMD:R_2512_6332Metric
- R37, R38, R39: value (none) -> 1k; footprint (none) -> Resistor_SMD:R_0603_1608Metric
- R46: value (none) -> 330; footprint (none) -> Resistor_SMD:R_0805_2012Metric
- R78, R79, R80, R81: value (none) -> 0; footprint (none) -> Resistor_SMD:R_0603_1608Metric
- U2: value (none) -> VCB4824SBO; footprint (none) -> interstate_footprints:VCB4824SB0-30WR3
- U6: value (none) -> LT1641-1; footprint (none) -> Package_SO:SOIC-8_3.9x4.9mm_P1.27mm
- U7: value (none) -> SN65HVD232; footprint (none) -> Package_SO:SOIC-8_3.9x4.9mm_P1.27mm
Connections:
- net ESC1_ADC1_UNFILT: now also U9.20 (PA4); no longer U9.23 (PA7)
- net ESC1_ADC2_UNFILT: now also U9.15 (PA1); no longer U9.26 (PB0)
- net ESC1_N: now also U9.17 (PA3); no longer U9.25 (PC5)
- net ESC1_ON: now also U9.14 (PA0); no longer U9.27 (PB1)
- net ESC1_P: now also U9.16 (PA2); no longer U9.24 (PC4)
- net ESC2_ADC1_UNFILT: now also U9.35 (PB14); no longer U9.15 (PA1)
- net ESC2_ADC2_UNFILT: now also U9.27 (PB1); no longer U9.20 (PA4)
- net ESC2_N: now also U9.30 (PB11); no longer U9.17 (PA3)
- net ESC2_ON: now also U9.36 (PB15); no longer U9.21 (PA5)
- net ESC2_P: now also U9.29 (PB10); no longer U9.16 (PA2)
- net ESC3_ADC1_UNFILT: now also U9.26 (PB0); no longer U9.35 (PB14)
- net ESC3_ADC2_UNFILT: now also U9.22 (PA6); no longer U9.36 (PB15)
- net ESC3_N: now also U9.25 (PC5); no longer U9.30 (PB11)
- net ESC3_ON: now also U9.21 (PA5); no longer U9.34 (PB13)
- net ESC3_P: now also U9.24 (PC4); no longer U9.29 (PB10)
- net GND: now also U1.1, U1.2, U1.4 (-), U1.5 (+), U1.6 (-), U1.7 (+); no longer U1.10 (-), U1.11 (+), U1.13, U1.14, U1.8 (-), U1.9 (+)
- net at R43.2: now also U1.8 (-); no longer U1.6 (-)
- net at R44.1: now also U1.13; no longer U1.2
- net at R41.2: now also U1.10 (-); no longer U1.4 (-)
- net at R40.2: now also U1.11 (+); no longer U1.5 (+)
- net at R42.2: now also U1.9 (+); no longer U1.7 (+)
- net at R45.1: now also U1.14; no longer U1.1

Commit message: finished routing v1?
Parts:
- added TP?: (no value), symbol Connector:TestPoint
- added TP? (x5): TestPoint, TestPoint:TestPoint_Pad_D1.0mm, symbol Connector:TestPoint
- U1: value (none) -> LM339
- U1: value (none) -> LM339; footprint (none) -> Package_SO:SOIC-14_3.9x8.7mm_P1.27mm
Connections:
- net ESC1_GND is gone; now on net GND: R54.1
- net ESC2_GND is gone; now on net GND: R61.1
- net ESC3_GND is gone; now on net GND: R68.1
- net +12V: now also TP?.1
- net +24V: now also TP?.1
- net BATT_GOOD: now also U9.43 (PA10)
- net ESTOP2: now also J3.3 (Pin_3); no longer J3.2 (Pin_2)
- net GND: now also J3.1 (Pin_1); no longer J3.4 (Pin_4)
- net LAMP1_ON: now also U9.4 (PC15)
- net LAMP2_ON: now also U9.3 (PC14)
- net LAMP3_ON: now also U9.2 (PC13)
- net LAMP4_ON: now also U9.62 (PB9)
- net LED1: now also U9.5 (PF0)
- net LED2: now also U9.6 (PF1)
- net SYS_ON: now also TP?.1
- net nESTOP1: now also TP?.1
- net nESTOP2: now also J3.2 (Pin_2), TP?.1; no longer J3.3 (Pin_3)
- net at R4.2, R5.2: now also J3.4 (Pin_4); no longer J3.1 (Pin_1)
- net at C30.1, R28.2, R29.1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: now also TP?.1
Other:
- moved on the sheet: C1, J3, R10, R11, R12, R4, R40, R41, R42, R43, R44, R45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

Commit message: ordered board + BOM
Parts:
- added PA15, PA7, PB4, PB5, PB7, TP7, TP8, TP9: TestPoint, TestPoint:TestPoint_Pad_D1.0mm, symbol Connector:TestPoint
- added PB3: (no value), TestPoint:TestPoint_Pad_D1.0mm, symbol Connector:TestPoint
- added SW2: (no value), symbol Switch:SW_SPDT
- C6: value ??nF -> (none); footprint Capacitor_SMD:C_0805_2012Metric -> (none); Digikey (none) -> 1292-1462-1-ND
- D2, D3: value RED -> (none); footprint LED_SMD:LED_0603_1608Metric -> (none); Digikey (none) -> 160-1445-1-ND
- Q5: value Q_NMOS_GDS -> (none); footprint Package_TO_SOT_SMD:TO-263-2 -> (none)
- R17: value ??? -> (none); footprint Resistor_SMD:R_0603_1608Metric -> (none); Digikey (none) -> A102282CT-ND; Power (none) -> 50mW
- R18: value ??? -> (none); footprint Resistor_SMD:R_0603_1608Metric -> (none); Digikey (none) -> 13-RT0603BRD071K35LCT-ND; Power (none) -> 1mW
- R26: value 10 -> (none); footprint Resistor_SMD:R_0603_1608Metric -> (none); Digikey (none) -> RMCF0603FT10R0CT-ND
- R28: value ??? -> (none); footprint Resistor_SMD:R_0603_1608Metric -> (none); Digikey (none) -> A102282CT-ND
- R29: value ??? -> (none); footprint Resistor_SMD:R_0603_1608Metric -> (none); Digikey (none) -> 13-RT0603BRD071K35LCT-ND
- R46, R47: value 330 -> (none); footprint Resistor_SMD:R_0805_2012Metric -> (none); Digikey (none) -> CR0603-JW-331ELFCT-ND
- R48: value 120 -> (none); footprint Resistor_SMD:R_0603_1608Metric -> (none); Digikey (none) -> A129677CT-ND
- SW1: value RST -> (none); footprint Button_Switch_SMD:SW_SPST_B3SL-1022P -> (none); Digikey (none) -> SW1104CT-ND
- TP5: renamed from TP?; value TestPoint -> (none)
- U4: value MCP1804x-3302xMT -> (none); footprint Package_TO_SOT_SMD:SOT-89-5 -> (none); Digikey MCP1804T-3302I/MTTR-ND -> MCP1804T-5002I/MTCT-ND
- U6: value LT1641-1 -> (none); footprint Package_SO:SOIC-8_3.9x4.9mm_P1.27mm -> (none)
- gave numbers to parts that had none: 5
Connections:
- net +12V: now also J2.1 (Pin_1); no longer R3.1
- net ESC1_ADC1: now also TP7.1
- net ESC2_ADC1: now also TP8.1
- net ESC3_ADC1: now also TP9.1
- net ESTOP2: now also J3.2 (Pin_2), R43.1, TP6.1; no longer J3.3 (Pin_3)
- net GND: now also R3.2, SW2.2 (B); no longer J2.2 (Pin_2)
- net SWDIO: now also U9.46 (PA13); no longer U9.50 (PA15)
- net SYS_ON: now also SW2.3 (C)
- net nESTOP2: now also J3.3 (Pin_3); no longer J3.2 (Pin_2), R42.1, TP6.1
- net at R11.2, R12.1, R8.2: now also R42.1; no longer R43.1
- net at R10.1, R9.2: now also R40.1; no longer R41.1
- net SPARE_SPI_MOSI: now reaches U9.23 (PA7)
- net SPARE_SPI_MOSI: now also PA7.1
- net SPARE_SPI_SCK: now reaches U9.55 (PB3)
- net SPARE_SPI_SCK: now also PB3.1
- net SPARE_SPI_MISO: now reaches U9.56 (PB4)
- net SPARE_SPI_MISO: now also PB4.1
- net SPARE_SPI_SEL: now reaches U9.57 (PB5)
- net SPARE_SPI_SEL: now also PB5.1
- net SPARE_I2C_SDA: now reaches U9.59 (PB7)
- net SPARE_I2C_SDA: now also PB7.1
- removed net nESTOP1: J2.1 (Pin_1), R3.2, R40.1, TP5.1
- new net ESTOP1: J2.2 (Pin_2), R3.1, R41.1, TP5.1
- new net SPARE_I2C_SCL: PA15.1, U9.50 (PA15)
- no-connect marks 27 -> 31
Other:
- note added: "Sense Resistor: I_limit = 47mV/Rsense FB Pin: Compared against 1.233V reference to pull PWRGOOD high Timer Pin: dv * (C/i) = dt 64nF capacitor is 1ms allowed charge time"
- note removed: "Sense Resistor: I_limit = 47mV/Rsense FB Pin: Compared against 1.233V reference to pull PWRGOOD high"
- moved on the sheet: C1, J2, J3, R10, R11, R12, R4, R40, R41, R42, R43, R44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
